File: laser-keyboard.kicad_pcb (KiCad board)
At the start: 2 copper layers, 9.1 x 18.3 mm, 160 parts, among them J1 Conn_01x04_Pin, SW01_2 SW_Push, SW01_3 SW_Push, SW01_4 SW_Push, SW01_5 SW_Push, SW01_6 SW_Push, SW01_7 SW_Push, SW01_8 SW_Push, SW02_2 SW_Push, SW02_3 SW_Push, SW02_4 SW_Push, SW02_5 SW_Push, SW02_6 SW_Push, SW02_7 SW_Push, SW02_8 SW_Push, SW03_2 SW_Push, SW03_3 SW_Push, SW03_4 SW_Push, SW03_5 SW_Push, SW03_6 SW_Push, SW03_7 SW_Push, SW04_2 SW_Push, SW04_3 SW_Push, SW04_4 SW_Push, SW04_5 SW_Push, SW04_7 SW_Push, SW05_1 SW_Push, SW05_2 SW_Push, SW05_3 SW_Push, SW05_4 SW_Push, SW05_5 SW_Push, SW05_6 SW_Push, SW05_7 SW_Push, SW05_8 SW_Push, SW06_1 SW_Push, SW06_2 SW_Push, SW06_4 SW_Push, SW06_5 SW_Push, SW06_6 SW_Push, SW06_7 SW_Push, SW06_8 SW_Push, SW07_2 SW_Push, SW07_3 SW_Push, SW07_4 SW_Push, SW07_5 SW_Push, SW07_6 SW_Push, SW07_7 SW_Push, SW07_8 SW_Push, SW08_1 EncSW, SW08_2 SW_Push, SW08_3 SW_Push, SW08_4 SW_Push, SW08_5 SW_Push, SW08_6 SW_Push, SW08_7 SW_Push, U1 ATmega32U4-M, U3 TPS73601DBV, U4 PMW3360DM-T2QU, U5 TPS73601DBV, Y1 16Mhz

Commit message: wip
Parts:
- removed REF** (x5): 1U, MX_Only:MXOnly-1U-Hotswap
- added LED1: SK6812MINI-E, SK6812MINI-E:SK6812MINIE, F.Cu at (408.7, 174.9)
- added LED10: SK6812MINI-E, SK6812MINI-E:SK6812MINIE, F.Cu at (183.7, 174.9)
- added LED11: SK6812MINI-E, SK6812MINI-E:SK6812MINIE, F.Cu at (158.7, 174.9)
- added LED12: SK6812MINI-E, SK6812MINI-E:SK6812MINIE, F.Cu at (133.7, 174.9)
- added LED13: SK6812MINI-E, SK6812MINI-E:SK6812MINIE, F.Cu at (133.7, 257.6)
- added LED14: SK6812MINI-E, SK6812MINI-E:SK6812MINIE, F.Cu at (158.7, 257.6)
- added LED15: SK6812MINI-E, SK6812MINI-E:SK6812MINIE, F.Cu at (183.7, 257.6)
- added LED16: SK6812MINI-E, SK6812MINI-E:SK6812MINIE, F.Cu at (208.7, 257.6)
- added LED17: SK6812MINI-E, SK6812MINI-E:SK6812MINIE, F.Cu at (233.7, 257.6)
- added LED18: SK6812MINI-E, SK6812MINI-E:SK6812MINIE, F.Cu at (258.7, 257.6)
- added LED19: SK6812MINI-E, SK6812MINI-E:SK6812MINIE, F.Cu at (283.7, 257.6)
- added LED2: SK6812MINI-E, SK6812MINI-E:SK6812MINIE, F.Cu at (383.7, 174.9)
- added LED20: SK6812MINI-E, SK6812MINI-E:SK6812MINIE, F.Cu at (308.7, 257.6)
- added LED21: SK6812MINI-E, SK6812MINI-E:SK6812MINIE, F.Cu at (333.7, 257.6)
- added LED22: SK6812MINI-E, SK6812MINI-E:SK6812MINIE, F.Cu at (358.7, 257.6)
- added LED3: SK6812MINI-E, SK6812MINI-E:SK6812MINIE, F.Cu at (358.7, 174.9)
- added LED4: SK6812MINI-E, SK6812MINI-E:SK6812MINIE, F.Cu at (333.7, 174.9)
- added LED5: SK6812MINI-E, SK6812MINI-E:SK6812MINIE, F.Cu at (308.7, 174.9)
- added LED6: SK6812MINI-E, SK6812MINI-E:SK6812MINIE, F.Cu at (283.7, 174.9)
- added LED7: SK6812MINI-E, SK6812MINI-E:SK6812MINIE, F.Cu at (258.7, 174.9)
- added LED8: SK6812MINI-E, SK6812MINI-E:SK6812MINIE, F.Cu at (233.7, 174.9)
- added LED9: SK6812MINI-E, SK6812MINI-E:SK6812MINIE, F.Cu at (208.7, 174.9)
- U4: moved to B.Cu
- moved D08_1 266.5 mm to (459.0, 254.3), turned to 90 degrees
- moved D08_2 243.3 mm to (435.2, 254.3), turned to 90 degrees
- moved D05_1 229.9 mm to (459.0, 187.6), turned to 90 degrees
- moved D08_3 224.6 mm to (416.2, 254.3), turned to 90 degrees
- moved D06_1 217.0 mm to (440.0, 187.6), turned to 90 degrees
- moved SW08_1 215.2 mm to (450.7, 257.1)
- moved D07_2 211.8 mm to (416.2, 235.2), turned to 90 degrees
- moved D08_4 205.9 mm to (397.1, 254.3), turned to 90 degrees
- moved D06_2 180.3 mm to (399.5, 211.4), turned to 90 degrees
- moved D07_3 180.0 mm to (385.2, 230.5), turned to 90 degrees
- moved D05_2 177.9 mm to (406.6, 192.3), turned to 90 degrees
- moved R2 177.9 mm to (271.2, 282.9)
- moved R5 177.9 mm to (271.2, 292.7)
- moved U3 177.9 mm to (263.3, 305.7)
- moved R10 177.9 mm to (265.6, 292.7)
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Routing:
- net DGND: track 38.7 -> 0.00 mm, vias 4 -> 0
- net DVCC: track 28.1 -> 0.00 mm, vias 2 -> 0
- net DD+: track 23.0 -> 0.00 mm, vias 2 -> 0
- net DGNDPWR: track 22.7 -> 0.00 mm
- net DD-: track 20.7 -> 0.00 mm, vias 2 -> 0
- net D+5V: track 9.60 -> 0.00 mm, vias 2 -> 0
- net Net-(DJ1-CC2): track 4.42 -> 0.00 mm
- net Net-(DJ1-CC1): track 4.26 -> 0.00 mm
Other:
- board size 9.1 x 18.3 mm -> 336.8 x 120.9 mm

Commit message: wip
Parts:
- moved R10 198.9 mm to (453.5, 227.5)
- moved U5 192.4 mm to (429.9, 219.6)
- moved R5 190.6 mm to (452.6, 234.1)
- moved U3 190.2 mm to (428.7, 211.8)
- moved R9 185.1 mm to (431.1, 206.7)
- moved C19 182.9 mm to (456.3, 221.8)
- moved C17 179.6 mm to (446.6, 201.3)
- moved R6 175.3 mm to (421.6, 205.9)
- moved C21 172.1 mm to (445.8, 231.7)
- moved C10 170.8 mm to (440.5, 201.1)
- moved R8 169.2 mm to (426.8, 234.6), turned to 0 degrees
- moved R7 168.1 mm to (422.6, 222.7)
- moved C16 163.9 mm to (435.4, 226.4)
- moved C14 163.2 mm to (442.7, 236.9)
- moved C20 158.5 mm to (434.7, 237.5)
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Connections:
- LED1 pad 1: Net-(LED1-VDD) -> +5V
- LED1 pad 3: Net-(LED1-GND) -> GND
- LED10 pad 1: Net-(LED1-VDD) -> +5V
- LED10 pad 3: Net-(LED1-GND) -> GND
- LED11 pad 1: Net-(LED1-VDD) -> +5V
- LED11 pad 3: Net-(LED1-GND) -> GND
- LED12 pad 1: Net-(LED1-VDD) -> +5V
- LED12 pad 3: Net-(LED1-GND) -> GND
- LED13 pad 1: Net-(LED1-VDD) -> +5V
- LED13 pad 3: Net-(LED1-GND) -> GND
- LED14 pad 1: Net-(LED1-VDD) -> +5V
- LED14 pad 3: Net-(LED1-GND) -> GND
- LED15 pad 1: Net-(LED1-VDD) -> +5V
- LED15 pad 3: Net-(LED1-GND) -> GND
- LED16 pad 1: Net-(LED1-VDD) -> +5V
- LED16 pad 3: Net-(LED1-GND) -> GND
- LED17 pad 1: Net-(LED1-VDD) -> +5V
- LED17 pad 3: Net-(LED1-GND) -> GND
- LED18 pad 1: Net-(LED1-VDD) -> +5V
- LED18 pad 3: Net-(LED1-GND) -> GND
- LED19 pad 1: Net-(LED1-VDD) -> +5V
- LED19 pad 3: Net-(LED1-GND) -> GND
- LED2 pad 1: Net-(LED1-VDD) -> +5V
- LED2 pad 3: Net-(LED1-GND) -> GND
- LED20 pad 1: Net-(LED1-VDD) -> +5V
- LED20 pad 3: Net-(LED1-GND) -> GND
- LED21 pad 1: Net-(LED1-VDD) -> +5V
- LED21 pad 3: Net-(LED1-GND) -> GND
- LED22 pad 1: Net-(LED1-VDD) -> +5V
- LED22 pad 2: Net-(LED22-DOUT) -> unconnected-(LED22-DOUT-Pad2)
- LED22 pad 3: Net-(LED1-GND) -> GND
- LED3 pad 1: Net-(LED1-VDD) -> +5V
- LED3 pad 3: Net-(LED1-GND) -> GND
- LED4 pad 1: Net-(LED1-VDD) -> +5V
- LED4 pad 3: Net-(LED1-GND) -> GND
- LED5 pad 1: Net-(LED1-VDD) -> +5V
- LED5 pad 3: Net-(LED1-GND) -> GND
- LED6 pad 1: Net-(LED1-VDD) -> +5V
- LED6 pad 3: Net-(LED1-GND) -> GND
- LED7 pad 1: Net-(LED1-VDD) -> +5V
- LED7 pad 3: Net-(LED1-GND) -> GND
- LED8 pad 1: Net-(LED1-VDD) -> +5V
- LED8 pad 3: Net-(LED1-GND) -> GND
- LED9 pad 1: Net-(LED1-VDD) -> +5V
- LED9 pad 3: Net-(LED1-GND) -> GND
Routing:
- net GND: track 0.00 -> 99.0 mm, vias 0 -> 6
- net +5V: track 0.00 -> 87.7 mm, vias 0 -> 6
- net RESET: track 0.00 -> 51.6 mm, vias 0 -> 4
- net D-: track 0.00 -> 24.5 mm, vias 0 -> 2
- net D+: track 0.00 -> 23.8 mm, vias 0 -> 2
- net Net-(U1-~{HWB}/PE2): track 0.00 -> 20.8 mm
- net Net-(U1-UCAP): track 0.00 -> 15.7 mm, vias 0 -> 2
- net Net-(D08_1-A): track 0.00 -> 13.8 mm
- net Net-(U1-XTAL2): track 0.00 -> 12.0 mm
- net Net-(U1-XTAL1): track 0.00 -> 11.5 mm
- net Net-(U1-D+): track 0.00 -> 10.5 mm
- net Net-(U1-D-): track 0.00 -> 10.2 mm, vias 0 -> 2

Commit message: wip
Parts:
- added REF**: breakaway-mousebites, random-keyboard-parts:breakaway-mousebites, F.Cu at (296.4, 167.5)
- added REF**: breakaway-mousebites, random-keyboard-parts:breakaway-mousebites, F.Cu at (296.4, 171.4)
- moved C17 31.7 mm to (444.9, 232.9), turned to -90 degrees
- moved C10 28.4 mm to (443.7, 229.3)
- moved R8 27.1 mm to (434.4, 208.7)
- moved R6 27.1 mm to (438.7, 226.8)
- moved C14 26.7 mm to (429.4, 213.8)
- moved C19 22.0 mm to (434.3, 221.3)
- moved C21 20.9 mm to (429.4, 218.8)
- moved U3 14.2 mm to (431.9, 225.6), turned to 0 degrees
- moved R7 13.2 mm to (429.4, 211.4)
- moved U5 12.4 mm to (429.4, 207.2), turned to -90 degrees
- moved R5 11.5 mm to (443.7, 226.9)
- moved DR1 11.2 mm to (289.7, 158.8)
- moved DR2 11.2 mm to (306.3, 154.0)
- moved DR3 11.2 mm to (306.3, 158.7)
- moved DC1 11.2 mm to (286.6, 158.7)
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Connections:
- LED11 pad 2: Net-(LED10-DIN) -> Net-(LED11-DOUT)
- LED11 pad 4: Net-(LED11-DIN) -> Net-(LED10-DOUT)
- LED12 pad 2: Net-(LED11-DIN) -> Net-(LED12-DOUT)
- LED12 pad 4: Net-(LED12-DIN) -> Net-(LED11-DOUT)
- LED13 pad 4: Net-(LED13-DIN) -> Net-(LED12-DOUT)
- LED3 pad 4: Net-(LED3-DIN) -> Net-(LED2-DOUT)
- LED4 pad 2: Net-(LED3-DIN) -> Net-(LED4-DOUT)
- LED4 pad 4: Net-(LED2-DOUT) -> Net-(LED3-DOUT)
- LED5 pad 2: Net-(LED12-DIN) -> Net-(LED5-DOUT)
- LED5 pad 4: Net-(LED5-DIN) -> Net-(LED4-DOUT)
- LED6 pad 2: Net-(LED5-DIN) -> Net-(LED6-DOUT)
- LED6 pad 4: Net-(LED3-DOUT) -> Net-(LED5-DOUT)
- LED7 pad 2: Net-(LED13-DIN) -> Net-(LED7-DOUT)
- LED7 pad 4: Net-(LED7-DIN) -> Net-(LED6-DOUT)
- LED8 pad 2: Net-(LED7-DIN) -> Net-(LED8-DOUT)
- LED8 pad 4: Net-(LED8-DIN) -> Net-(LED7-DOUT)
- LED9 pad 2: Net-(LED8-DIN) -> Net-(LED10-DIN)
- LED9 pad 4: Net-(LED10-DOUT) -> Net-(LED8-DOUT)
- U1 pad 18: col03 -> row08
- U1 pad 19: col04 -> row04
- U1 pad 20: col05 -> col02
- U1 pad 21: col06 -> unconnected-(U1-PD3-Pad21)
- U1 pad 22: col08 -> col07
- U1 pad 25: col07 -> col03
- U1 pad 26: row01 -> col04
- U1 pad 27: row02 -> col05
- U1 pad 28: row08 -> col06
- U1 pad 29: row07 -> row01
- U1 pad 30: unconnected-(U1-PB6-Pad30) -> row02
- U1 pad 31: col01 -> row03
- U1 pad 32: col02 -> row05
- U1 pad 36: row06 -> col08
- U1 pad 37: row05 -> col01
- U1 pad 38: row04 -> row06
- U1 pad 39: row03 -> row07
Routing:
- net GND: track 99.0 -> 935.8 mm, vias 6 -> 13
- net +5V: track 87.7 -> 914.0 mm, vias 6 -> 21
- net col02: track 0.00 -> 592.8 mm, vias 0 -> 6
- net col03: track 0.00 -> 518.6 mm, vias 0 -> 8
- net col04: track 0.00 -> 457.5 mm, vias 0 -> 9
- net col05: track 0.00 -> 361.5 mm, vias 0 -> 9
- net col01: track 0.00 -> 324.4 mm, vias 0 -> 2
- net col06: track 0.00 -> 279.9 mm, vias 0 -> 8
- net SCLK: track 0.00 -> 261.5 mm, vias 0 -> 2
- net MOSI: track 0.00 -> 253.0 mm, vias 0 -> 3
- net MOTION: track 0.00 -> 252.5 mm, vias 0 -> 5
- net MISO: track 0.00 -> 246.6 mm, vias 0 -> 1
- net NCS: track 0.00 -> 243.4 mm, vias 0 -> 3
- net row05: track 0.00 -> 232.8 mm, vias 0 -> 2
- net col07: track 0.00 -> 231.3 mm, vias 0 -> 10
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- added copper zone on B.Cu, net (none)
- added copper zone on F.Cu, net (none)
Other:
- board size 336.8 x 120.9 mm -> 336.8 x 109.9 mm

Commit message: pos, bom, gerbers
Connections:
- SW01_2 pad 1: col02 -> col01
- SW01_3 pad 1: col03 -> col02
- SW01_4 pad 1: col04 -> col03
- SW01_5 pad 1: col05 -> col04
- SW01_6 pad 1: col06 -> col05
- SW01_7 pad 1: col07 -> col06
- SW01_8 pad 1: col08 -> col07
- SW02_2 pad 1: col02 -> col01
- SW02_3 pad 1: col03 -> col02
- SW02_4 pad 1: col04 -> col03
- SW02_5 pad 1: col05 -> col04
- SW02_6 pad 1: col06 -> col05
- SW02_7 pad 1: col07 -> col06
- SW02_8 pad 1: col08 -> col07
- SW03_2 pad 1: col02 -> col01
- SW03_3 pad 1: col03 -> col02
- SW03_4 pad 1: col04 -> col03
- SW03_5 pad 1: col05 -> col04
- SW03_6 pad 1: col06 -> col05
- SW03_7 pad 1: col07 -> col06
- SW04_2 pad 1: col02 -> col01
- SW04_3 pad 1: col03 -> col02
- SW04_4 pad 1: col04 -> col03
- SW04_5 pad 1: col05 -> col04
- SW04_7 pad 1: col07 -> col06
- SW05_1 pad 1: col01 -> col08
- SW05_2 pad 1: col02 -> col01
- SW05_3 pad 1: col03 -> col02
- SW05_4 pad 1: col04 -> col03
- SW05_5 pad 1: col05 -> col04
- SW05_6 pad 1: col06 -> col05
- SW05_7 pad 1: col07 -> col06
- SW05_8 pad 1: col08 -> col07
- SW06_1 pad 1: col01 -> col08
- SW06_2 pad 1: col02 -> col01
- SW06_4 pad 1: col04 -> col03
- SW06_5 pad 1: col05 -> col04
- SW06_6 pad 1: col06 -> col05
- SW06_7 pad 1: col07 -> col06
- SW06_8 pad 1: col08 -> col07
- SW07_2 pad 1: col02 -> col01
- SW07_3 pad 1: col03 -> col02
- SW07_4 pad 1: col04 -> col03
- SW07_5 pad 1: col05 -> col04
- SW07_6 pad 1: col06 -> col05
- SW07_7 pad 1: col07 -> col06
- SW07_8 pad 1: col08 -> col07
- SW08_1 pad S2: col01 -> col08
- SW08_2 pad 1: col02 -> col01
- SW08_3 pad 1: col03 -> col02
- SW08_4 pad 1: col04 -> col03
- SW08_5 pad 1: col05 -> col04
- SW08_6 pad 1: col06 -> col05
- SW08_7 pad 1: col07 -> col06
- U1 pad 20: col02 -> col01
- U1 pad 22: col07 -> col06
- U1 pad 25: col03 -> col02
- U1 pad 26: col04 -> col03
- U1 pad 27: col05 -> col04
- U1 pad 28: col06 -> col05
- U1 pad 36: col08 -> col07
- U1 pad 37: col01 -> col08
Routing:
- net col01: track 324.4 -> 592.8 mm, vias 2 -> 6
- net col08: track 106.7 -> 324.4 mm, vias 3 -> 2
- net col07: track 231.3 -> 106.7 mm, vias 10 -> 3
- net col04: track 457.5 -> 361.5 mm
- net col05: track 361.5 -> 279.9 mm, vias 9 -> 8
- net col02: track 592.8 -> 518.6 mm, vias 6 -> 8
- net col03: track 518.6 -> 457.5 mm, vias 8 -> 9
- net col06: track 279.9 -> 231.3 mm, vias 8 -> 10
