File: laser-keyboard.kicad_pcb (KiCad board)
At the start: 2 copper layers, 336.8 x 109.9 mm, 179 parts, among them J1 Conn_01x04_Pin, SW01_2 SW_Push, SW01_3 SW_Push, SW01_4 SW_Push, SW01_5 SW_Push, SW01_6 SW_Push, SW01_7 SW_Push, SW01_8 SW_Push, SW02_2 SW_Push, SW02_3 SW_Push, SW02_4 SW_Push, SW02_5 SW_Push, SW02_6 SW_Push, SW02_7 SW_Push, SW02_8 SW_Push, SW03_2 SW_Push, SW03_3 SW_Push, SW03_4 SW_Push, SW03_5 SW_Push, SW03_6 SW_Push, SW03_7 SW_Push, SW04_2 SW_Push, SW04_3 SW_Push, SW04_4 SW_Push, SW04_5 SW_Push, SW04_7 SW_Push, SW05_1 SW_Push, SW05_2 SW_Push, SW05_3 SW_Push, SW05_4 SW_Push, SW05_5 SW_Push, SW05_6 SW_Push, SW05_7 SW_Push, SW05_8 SW_Push, SW06_1 SW_Push, SW06_2 SW_Push, SW06_4 SW_Push, SW06_5 SW_Push, SW06_6 SW_Push, SW06_7 SW_Push, SW06_8 SW_Push, SW07_2 SW_Push, SW07_3 SW_Push, SW07_4 SW_Push, SW07_5 SW_Push, SW07_6 SW_Push, SW07_7 SW_Push, SW07_8 SW_Push, SW08_1 EncSW, SW08_2 SW_Push, SW08_3 SW_Push, SW08_4 SW_Push, SW08_5 SW_Push, SW08_6 SW_Push, SW08_7 SW_Push, U1 ATmega32U4-M, U3 TPS73601DBV, U4 PMW3360DM-T2QU, U5 TPS73601DBV, Y1 16Mhz

Commit message: Replace out-of-stock JLCPCB parts and sync LCSC numbers
- R7 52.3k: C229694 -> C488889 (Yageo RC1206FR-0752K3L)
- R6 63.4k: C159496 -> C488931 (Yageo RC1206FR-0763K4L)
- DF1: C2833485 (0805 fuse on 1206 footprint) -> C883124 (BHFUSE BSMD1206-050-16V, 1206)
- Sync schematic LCSC fields with bom.csv (R3-R9, DR1-DR3, DF1)
- Update PCB from schematic; project re-saved in KiCad 10 format

Co-Authored-By: Claude Opus 5.5 <noreply@anthropic.com>
Parts:
- DF1: value SMD0805-050-16V -> BSMD1206-050-16V
