File: laser-keyboard.kicad_sch (KiCad schematic)
At the start: 155 parts, among them J1 Conn_01x04_Pin, SW01_2 SW_Push, SW01_3 SW_Push, SW01_4 SW_Push, SW01_5 SW_Push, SW01_6 SW_Push, SW01_7 SW_Push, SW01_8 SW_Push, SW02_2 SW_Push, SW02_3 SW_Push, SW02_4 SW_Push, SW02_5 SW_Push, SW02_6 SW_Push, SW02_7 SW_Push, SW02_8 SW_Push, SW03_2 SW_Push, SW03_3 SW_Push, SW03_4 SW_Push, SW03_5 SW_Push, SW03_6 SW_Push, SW03_7 SW_Push, SW04_2 SW_Push, SW04_3 SW_Push, SW04_4 SW_Push, SW04_5 SW_Push, SW04_7 SW_Push, SW05_1 SW_Push, SW05_2 SW_Push, SW05_3 SW_Push, SW05_4 SW_Push, SW05_5 SW_Push, SW05_6 SW_Push, SW05_7 SW_Push, SW05_8 SW_Push, SW06_1 SW_Push, SW06_2 SW_Push, SW06_4 SW_Push, SW06_5 SW_Push, SW06_6 SW_Push, SW06_7 SW_Push, SW06_8 SW_Push, SW07_2 SW_Push, SW07_3 SW_Push, SW07_4 SW_Push, SW07_5 SW_Push, SW07_6 SW_Push, SW07_7 SW_Push, SW07_8 SW_Push, SW08_1 EncSW, SW08_2 SW_Push, SW08_3 SW_Push, SW08_4 SW_Push, SW08_5 SW_Push, SW08_6 SW_Push, SW08_7 SW_Push, U1 ATmega32U4-M, U3 TPS73601DBV, U4 PMW3360DM-T2QU, U5 TPS73601DBV, Y1 16Mhz

Commit message: v1.0.0
Parts:
- added LED1, LED10, LED11, LED12, LED13, LED14, LED15, LED16, LED17, LED18, LED19, LED2, LED20, LED21, LED22, LED3, LED4, LED5, LED6, LED7, LED8, LED9: SK6812MINI-E, SK6812MINI-E:SK6812MINIE, symbol SK6812MINI-E:SK6812MINI-E
- DJ1: value USB_C_Receptacle_USB2.0 -> USB_C_Receptacle_USB2.0_16P; symbol Connector:USB_C_Receptacle_USB2.0 -> Connector:USB_C_Receptacle_USB2.0_16P
- DJ2, J1: footprint (none) -> 1157-04AU:FPC-SMD_4P-P1.00_1157-04AU; symbol Connector:Conn_01x04_Pin -> 1157-04AU:1157-04AU; LCSC Part (none) -> C2886699
- SW01_2: footprint MX_Only:MXOnly-1U-Hotswap -> MX_Only:MXOnly-1.5U-Hotswap
- SW02_2, SW07_3: footprint MX_Only:MXOnly-1U-Hotswap -> MX_Only:MXOnly-1.75U-Hotswap
- SW03_2, SW06_2: footprint MX_Only:MXOnly-1U-Hotswap -> MX_Only:MXOnly-2.25U-Hotswap
- SW04_2: footprint MX_Only:MXOnly-2.25U-Hotswap -> MX_Only:MXOnly-1.25U-Hotswap
- SW04_3, SW04_4, SW04_7, SW08_5, SW08_6: footprint MX_Only:MXOnly-1U-Hotswap -> MX_Only:MXOnly-1.25U-Hotswap
- SW04_5: footprint MX_Only:MXOnly-1U-Hotswap -> MX_Only:MXOnly-2.25U-Hotswap-ReversedStabilizers
- SW05_1: footprint MX_Only:MXOnly-2U-Hotswap -> MX_Only:MXOnly-1U-Hotswap
- SW05_2: footprint MX_Only:MXOnly-2U-Hotswap -> MX_Only:MXOnly-1.5U-Hotswap
- SW08_3: footprint MX_Only:MXOnly-2.75U-Hotswap -> MX_Only:MXOnly-1U-Hotswap
- SW08_7: footprint MX_Only:MXOnly-1U-Hotswap -> MX_Only:MXOnly-2.75U-Hotswap-ReversedStabilizers
- U4: footprint PMW3360DM-T2QU:PMW3360 -> KiCad:PMW3360
Connections:
- net +5V: now also J1.1, LED1.1 (VDD), LED10.1 (VDD), LED11.1 (VDD), LED12.1 (VDD), LED13.1 (VDD), LED14.1 (VDD), LED15.1 (VDD), LED16.1 (VDD), LED17.1 (VDD), LED18.1 (VDD), LED19.1 (VDD), LED2.1 (VDD), LED20.1 (VDD), LED21.1 (VDD), LED22.1 (VDD), LED3.1 (VDD), LED4.1 (VDD), LED5.1 (VDD), LED6.1 (VDD), LED7.1 (VDD), LED8.1 (VDD), LED9.1 (VDD); no longer J1.4 (Pin_4)
- net D+: now also J1.4; no longer J1.1 (Pin_1)
- net D+5V: now also DJ2.4; no longer DJ2.1 (Pin_1)
- net D-: now also J1.3; no longer J1.2 (Pin_2)
- net DD+: now also DJ2.1; no longer DJ2.4 (Pin_4)
- net DD-: now also DJ2.2; no longer DJ2.3 (Pin_3)
- net DGND: now also DJ2.3; no longer DJ2.2 (Pin_2)
- net GND: now also J1.2, LED1.3 (GND), LED10.3 (GND), LED11.3 (GND), LED12.3 (GND), LED13.3 (GND), LED14.3 (GND), LED15.3 (GND), LED16.3 (GND), LED17.3 (GND), LED18.3 (GND), LED19.3 (GND), LED2.3 (GND), LED20.3 (GND), LED21.3 (GND), LED22.3 (GND), LED3.3 (GND), LED4.3 (GND), LED5.3 (GND), LED6.3 (GND), LED7.3 (GND), LED8.3 (GND), LED9.3 (GND); no longer J1.3 (Pin_3)
- net LED: now also LED1.4 (DIN)
- net col01: now also SW01_2.1, SW02_2.1, SW03_2.1, SW04_2.1, SW05_2.1, SW06_2.1, SW07_2.1, SW08_2.1, U1.20 (PD2); no longer SW05_1.1, SW06_1.1, SW08_1.S2, U1.31 (PC6)
- net col02: now also SW01_3.1, SW02_3.1, SW03_3.1, SW04_3.1, SW05_3.1, SW07_3.1, SW08_3.1, U1.25 (PD4); no longer SW01_2.1, SW02_2.1, SW03_2.1, SW04_2.1, SW05_2.1, SW06_2.1, SW07_2.1, SW08_2.1, U1.32 (PC7)
- net col03: now also SW01_4.1, SW02_4.1, SW03_4.1, SW04_4.1, SW05_4.1, SW06_4.1, SW07_4.1, SW08_4.1, U1.26 (PD6); no longer SW01_3.1, SW02_3.1, SW03_3.1, SW04_3.1, SW05_3.1, SW07_3.1, SW08_3.1, U1.18 (PD0)
- net col04: now also SW01_5.1, SW02_5.1, SW03_5.1, SW04_5.1, SW05_5.1, SW06_5.1, SW07_5.1, SW08_5.1, U1.27 (PD7); no longer SW01_4.1, SW02_4.1, SW03_4.1, SW04_4.1, SW05_4.1, SW06_4.1, SW07_4.1, SW08_4.1, U1.19 (PD1)
- net col05: now also SW01_6.1, SW02_6.1, SW03_6.1, SW05_6.1, SW06_6.1, SW07_6.1, SW08_6.1, U1.28 (PB4); no longer SW01_5.1, SW02_5.1, SW03_5.1, SW04_5.1, SW05_5.1, SW06_5.1, SW07_5.1, SW08_5.1, U1.20 (PD2)
- net col06: now also SW01_7.1, SW02_7.1, SW03_7.1, SW04_7.1, SW05_7.1, SW06_7.1, SW07_7.1, SW08_7.1, U1.22 (PD5); no longer SW01_6.1, SW02_6.1, SW03_6.1, SW05_6.1, SW06_6.1, SW07_6.1, SW08_6.1, U1.21 (PD3)
- net col07: now also SW01_8.1, SW02_8.1, SW05_8.1, SW06_8.1, SW07_8.1, U1.36 (PF7); no longer SW01_7.1, SW02_7.1, SW03_7.1, SW04_7.1, SW05_7.1, SW06_7.1, SW07_7.1, SW08_7.1, U1.25 (PD4)
- net col08: now also SW05_1.1, SW06_1.1, SW08_1.S2, U1.37 (PF6); no longer SW01_8.1, SW02_8.1, SW05_8.1, SW06_8.1, SW07_8.1, U1.22 (PD5)
- net row01: now also U1.29 (PB5); no longer U1.26 (PD6)
- net row02: now also U1.30 (PB6); no longer U1.27 (PD7)
- net row03: now also U1.31 (PC6); no longer U1.39 (PF4)
- net row04: now also U1.19 (PD1); no longer U1.38 (PF5)
- net row05: now also U1.32 (PC7); no longer U1.37 (PF6)
- net row06: now also U1.38 (PF5); no longer U1.36 (PF7)
- net row07: now also U1.39 (PF4); no longer U1.29 (PB5)
- net row08: now also U1.18 (PD0); no longer U1.28 (PB4)
- new net: LED4.2 (DOUT), LED5.4 (DIN)
- new net: LED3.2 (DOUT), LED4.4 (DIN)
- new net: LED12.2 (DOUT), LED13.4 (DIN)
- new net: LED11.2 (DOUT), LED12.4 (DIN)
- new net: LED5.2 (DOUT), LED6.4 (DIN)
- new net: LED16.2 (DOUT), LED17.4 (DIN)
- new net: LED15.2 (DOUT), LED16.4 (DIN)
- new net: LED2.2 (DOUT), LED3.4 (DIN)
- new net: LED1.2 (DOUT), LED2.4 (DIN)
- new net: LED10.2 (DOUT), LED11.4 (DIN)
- new net: LED8.2 (DOUT), LED9.4 (DIN)
- new net: LED7.2 (DOUT), LED8.4 (DIN)
- new net: LED14.2 (DOUT), LED15.4 (DIN)
- new net: LED13.2 (DOUT), LED14.4 (DIN)
- new net: LED10.4 (DIN), LED9.2 (DOUT)
- new net: LED6.2 (DOUT), LED7.4 (DIN)
- new net: LED19.2 (DOUT), LED20.4 (DIN)
- new net: LED18.2 (DOUT), LED19.4 (DIN)
- new net: LED20.2 (DOUT), LED21.4 (DIN)
- new net: LED21.2 (DOUT), LED22.4 (DIN)
- new net: LED17.2 (DOUT), LED18.4 (DIN)
- no-connect marks 9 -> 14
Other:
- note added: "LED"
- moved on the sheet: C10, C11, C12, C13, C14, C15, C16, C17, C18, C19, C20, C21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
