File: laser-keyboard.kicad_sch (KiCad schematic)
At the start: 177 parts, among them J1 Conn_01x04_Pin, SW01_2 SW_Push, SW01_3 SW_Push, SW01_4 SW_Push, SW01_5 SW_Push, SW01_6 SW_Push, SW01_7 SW_Push, SW01_8 SW_Push, SW02_2 SW_Push, SW02_3 SW_Push, SW02_4 SW_Push, SW02_5 SW_Push, SW02_6 SW_Push, SW02_7 SW_Push, SW02_8 SW_Push, SW03_2 SW_Push, SW03_3 SW_Push, SW03_4 SW_Push, SW03_5 SW_Push, SW03_6 SW_Push, SW03_7 SW_Push, SW04_2 SW_Push, SW04_3 SW_Push, SW04_4 SW_Push, SW04_5 SW_Push, SW04_7 SW_Push, SW05_1 SW_Push, SW05_2 SW_Push, SW05_3 SW_Push, SW05_4 SW_Push, SW05_5 SW_Push, SW05_6 SW_Push, SW05_7 SW_Push, SW05_8 SW_Push, SW06_1 SW_Push, SW06_2 SW_Push, SW06_4 SW_Push, SW06_5 SW_Push, SW06_6 SW_Push, SW06_7 SW_Push, SW06_8 SW_Push, SW07_2 SW_Push, SW07_3 SW_Push, SW07_4 SW_Push, SW07_5 SW_Push, SW07_6 SW_Push, SW07_7 SW_Push, SW07_8 SW_Push, SW08_1 EncSW, SW08_2 SW_Push, SW08_3 SW_Push, SW08_4 SW_Push, SW08_5 SW_Push, SW08_6 SW_Push, SW08_7 SW_Push, U1 ATmega32U4-M, U3 TPS73601DBV, U4 PMW3360DM-T2QU, U5 TPS73601DBV, Y1 16Mhz

Commit message: Replace out-of-stock JLCPCB parts and sync LCSC numbers
- R7 52.3k: C229694 -> C488889 (Yageo RC1206FR-0752K3L)
- R6 63.4k: C159496 -> C488931 (Yageo RC1206FR-0763K4L)
- DF1: C2833485 (0805 fuse on 1206 footprint) -> C883124 (BHFUSE BSMD1206-050-16V, 1206)
- Sync schematic LCSC fields with bom.csv (R3-R9, DR1-DR3, DF1)
- Update PCB from schematic; project re-saved in KiCad 10 format

Co-Authored-By: Claude Opus 5.5 <noreply@anthropic.com>
Parts:
- DF1: value SMD0805-050-16V -> BSMD1206-050-16V; LCSC C2833485 -> C883124; Manufacturer TECHFUSE -> BHFUSE; Manufacturer Part Number SMD0805-050-16V -> BSMD1206-050-16V; Package F0805 -> 1206
- DR1, DR2: LCSC C964991 -> C26033
- DR3: LCSC C2759631 -> C17927
- R3, R4, R9: LCSC C17928 -> C1489
- R5: LCSC C247280 -> C229581
- R6: LCSC C45027 -> C488931
- R7: LCSC C247238 -> C488889
- R8: LCSC C425547 -> C311945
Changed lines of the file:
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@@
 			)
 		)
-		(property "LCSC" "C964991"
+		(property "LCSC" "C26033"
 			(at 76.2 208.28 90)
 			(effects
@@
 			)
 		)
-		(property "LCSC" "C247280"
+		(property "LCSC" "C229581"
 			(at 283.21 288.29 90)
 			(effects
@@
 			)
 		)
-		(property "LCSC" "C425547"
+		(property "LCSC" "C311945"
 			(at 373.38 292.1 90)
 			(effects
@@
 			)
 		)
-		(property "LCSC" "C45027"
+		(property "LCSC" "C488931"
 			(at 295.91 292.1 90)
 			(effects
@@
 			)
 		)
-		(property "LCSC" "C247238"
+		(property "LCSC" "C488889"
 			(at 360.68 288.29 90)
 			(effects
@@
 			)
 		)
-		(property "LCSC" "C2759631"
+		(property "LCSC" "C17927"
 			(at 39.37 300.99 90)
 			(effects
@@
 			)
 		)
-		(property "Value" "SMD0805-050-16V"
+		(property "Value" "BSMD1206-050-16V"
 			(at 74.93 297.18 90)
 			(effects
@@
 			)
 		)
-		(property "Manufacturer" "TECHFUSE"
+		(property "Manufacturer" "BHFUSE"
 			(at 74.93 300.99 0)
 			(effects
@@
 			)
 		)
-		(property "Manufacturer Part Number" "SMD0805-050-16V"
+		(property "Manufacturer Part Number" "BSMD1206-050-16V"
 			(at 74.93 300.99 0)
 			(effects
@@
 			)
 		)
-		(property "LCSC" "C2833485"
+		(property "LCSC" "C883124"
 			(at 74.93 300.99 0)
 			(effects
@@
 			)
 		)
-		(property "Package" "F0805"
+		(property "Package" "1206"
 			(at 74.93 300.99 0)
 			(effects
@@
 			)
 		)
-		(property "LCSC" "C964991"
+		(property "LCSC" "C26033"
 			(at 76.2 210.82 90)
 			(effects
@@
 			)
 		)
-		(property "LCSC" "C17928"
+		(property "LCSC" "C1489"
 			(at 86.36 118.11 90)
 			(effects
@@
 			)
 		)
-		(property "LCSC" "C17928"
+		(property "LCSC" "C1489"
 			(at 289.56 252.73 90)
 			(effects
@@
 			)
 		)
-		(property "LCSC" "C17928"
+		(property "LCSC" "C1489"
 			(at 119.38 83.82 90)
 			(effects
