File: plate/plate.kicad_pcb (KiCad board)
At the start: 2 copper layers, 349 x 101.3 mm, 0 parts

Commit message: Update plate design, gerbers, foam svg, and gitignore
Other:
- board size 349 x 101.3 mm -> 346.8 x 99.1 mm
